Commit message: Ros progress

File: src/my_r2d2/r2d2.urdf.xacro (robot description, xacro)
@@ -1,4 +1,4 @@
 <?xml version="1.0"?>
-<robot name="visual">
+<robot xmlns:xacro="http://www.ros.org/wiki/xacro" name="robot_description">
   <material name="blue">
     <color rgba="0 0 0.8 1"/>
@@ -10,31 +10,61 @@
     <color rgba="1 1 1 1"/>
   </material>
-  <link name="base_link">
-    <visual>
-      <geometry>
-        <cylinder length="0.6" radius="0.2"/>
-      </geometry>
-      <material name="blue"/>
-    </visual>
-	<collision>
-      <geometry>
-        <cylinder length="0.6" radius="0.2"/>
-      </geometry>
+<xacro:property name="width" value="0.2" />
+<xacro:property name="bodylen" value="0.6" />
+<xacro:property name="leglen" value="0.6"/>
+<xacro:macro name="default_inertial" params="mass">
+        <inertial>
+                <mass value="${mass}" />
+                <inertia ixx="1.0" ixy="0.0" ixz="0.0"
+                     iyy="1.0" iyz="0.0"
+                     izz="1.0" />
+        </inertial>
+    </xacro:macro>
+<link name="base_footprint">
+</link>
+<joint name="base_joint" type="fixed">
+	<origin xyz="0 0 0.47"/>
+	<parent link="base_footprint"/>
+	<child link="base_link"/>
+</joint>
+<link name="base_link">
+    <visual>
+        <geometry>
+            <cylinder radius="${width}" length="${bodylen}"/>
+        </geometry>
+        <material name="blue"/>
+    </visual>
+    <collision>
+        <geometry>
+            <cylinder radius="${width}" length="${bodylen}"/>
+        </geometry>
     </collision>
-  </link>
-  <link name="right_leg">
-    <visual>
-      <geometry>
-        <box size="0.6 0.1 0.2"/>
-      </geometry>
-      <origin rpy="0 1.57075 0" xyz="0 0 -0.3"/>
-      <material name="white"/>
-    </visual>
-  </link>
-  <joint name="base_to_right_leg" type="fixed">
-    <parent link="base_link"/>
-    <child link="right_leg"/>
-    <origin xyz="0 -0.22 0.25"/>
-  </joint>
+</link>
+<xacro:macro name="leg" params="prefix reflect">
+    <link name="${prefix}_leg">
+        <visual>
+            <geometry>
+                <box size="${leglen} 0.1 0.2"/>
+            </geometry>
+            <origin xyz="0 0 -${leglen/2}" rpy="0 ${pi/2} 0"/>
+            <material name="white"/>
+        </visual>
+        <collision>
+            <geometry>
+                <box size="${leglen} 0.1 0.2"/>
+            </geometry>
+            <origin xyz="0 0 -${leglen/2}" rpy="0 ${pi/2} 0"/>
+        </collision>
+        <xacro:default_inertial mass="10"/>
+    </link>
+    <joint name="base_to_${prefix}_leg" type="fixed">
+        <parent link="base_link"/>
+        <child link="${prefix}_leg"/>
+        <origin xyz="0 ${reflect*(width+.02)} 0.25" />
+    </joint>
+    <!-- A bunch of stuff cut -->
+</xacro:macro>
+<xacro:leg prefix="right" reflect="1" />
+<xacro:leg prefix="left" reflect="-1" />
   <link name="right_base">
     <visual>
@@ -80,18 +110,4 @@
     <origin rpy="0 0 0" xyz="-0.133333333333 0 -0.085"/>
 	<axis xyz="0 0 1"/>
-  </joint>
-  <link name="left_leg">
-    <visual>
-      <geometry>
-        <box size="0.6 0.1 0.2"/>
-      </geometry>
-      <origin rpy="0 1.57075 0" xyz="0 0 -0.3"/>
-      <material name="white"/>
-    </visual>
-  </link>
-  <joint name="base_to_left_leg" type="fixed">
-    <parent link="base_link"/>
-    <child link="left_leg"/>
-    <origin xyz="0 0.22 0.25"/>
   </joint>
   <link name="left_base">
@@ -225,5 +241,5 @@
         <box size="0.08 0.08 0.08"/>
       </geometry>
-      <material name="blue"/>
+	<material name="blue"/>
     </visual>
   </link>
@@ -231,5 +247,27 @@
     <parent link="head"/>
     <child link="box"/>
-    <origin xyz="0.1814 0 0.1414"/>
-  </joint>
+    <origin xyz="0.15 0 0.11"/>
+  </joint>
+ <link name="lense">
+    <visual>
+	<material name="black"/>
+	 <geometry>
+        <sphere radius="0.02"/>
+      </geometry>
+    </visual>
+  </link>
+ <joint name="boxtolense" type="fixed">
+  <origin xyz="0.035 0 0"/>
+    <parent link="box"/>
+    <child link="lense"/>
+  </joint>
+  <joint name="lensetoeye" type="fixed">
+    <parent link="lense"/>
+    <child link="eye"/>
+    <origin rpy="-1.57075 0  -1.57075" xyz="0 0 0"/>
+  </joint>
+  <link name="eye">
+	 <visual>
+    </visual>
+  </link>
 </robot>
